Commit message: Optimized the robot model in Gazebo, now the wheel collision is a cylinder Fixed kinect support inertia, now intertia is insignificant

File: atom2_common/atom2_description/urdf/accesories/kinect_support.urdf.xacro (robot description, xacro)
@@ -15,10 +15,9 @@
         </geometry>
         </visual>
-        <inertial>
-        <mass value="0.1" />
+      <inertial>
+        <mass value="1e-5" />
         <origin xyz="0 0 0" rpy="0 0 0"/>
-        <box_inertia m="0.1" x="0.1" y="0.1" z="0.1" />
         <inertia ixx="1e-6" ixy="0" ixz="0" iyy="1e-6" iyz="0" izz="1e-6" />
-        </inertial>
+      </inertial>
     </link>
     <joint name="${prefix}_joint" type="fixed">

File: atom2_common/atom2_description/urdf/wheels/rubber_wheel.urdf.xacro (robot description, xacro)
@@ -44,7 +44,8 @@
       </visual>
       <collision>
-        <origin xyz="0 0 0" rpy="0 0 0" />
+        <origin xyz="0 0 0" rpy="1.57079632679 0 0" />
         <geometry>
-          <mesh_selector wheel = "${prefix}" extension = "_simple.stl" />
+          <!-- <mesh_selector wheel = "${prefix}" extension = "_simple.stl" /> -->
+          <cylinder length="0.04" radius="0.082"/>
         </geometry>
       </collision>
