Commit message: Fixed inverted frame bug

File: atom2_common/atom2_description/urdf/accesories/kinect.urdf.xacro (robot description, xacro)
@@ -68,5 +68,5 @@
           (Hence, don't publish them additionally!) -->
     <joint name="${prefix}_depth_joint" type="fixed">
-      <origin xyz="0 ${2 * -cam_py} 0" rpy="0 0 0" />
+      <!-- <origin xyz="0 ${2 * -cam_py} 0" rpy="0 0 0" /> -->
       <parent link="${prefix}_rgb_base_link" />
       <child link="${prefix}_depth_link" />
