Commit message: Deleted jaco and ur3 arm

File: atom2_common/atom2_description/robots/atom2_std.urdf.xacro (robot description, xacro)
@@ -103,27 +103,4 @@
   </xacro:if>
 <!-- - - - - - - - - - - - - - UR3 ARM IMPLEMENTATION  - - - - - - - - - - - - - -->
-<!--
-  <xacro:include filename="$(find ur_description)/urdf/ur3.urdf.xacro" />
-    <xacro:ur3_robot prefix="arm_"  joint_limited="true"
-			shoulder_pan_lower_limit="-3.14" shoulder_pan_upper_limit="3.14"
-			wrist_3_lower_limit="3.14" wrist_3_upper_limit="3.14"
-      transmission_hw_interface= "hardware_interface/PositionJointInterface" >
-    </xacro:ur3_robot>
-    <joint name="arm_base_joint" type="fixed">
-		<origin xyz="-0.23 0 0.21275" rpy="0 0 0" />
-		<parent link="atom2_base_link" />
-		<child link="arm_base_link" />
-	  </joint>
--->
-<!--
-<link name="root"/>
-    <joint name="arm_base_joint" type="fixed">
-		<origin xyz="0 0 0.21275" rpy="0 0 0" />
-		<parent link="atom2_base_link" />
-		<child link="root" />
-	  </joint>
- <xacro:include filename="$(find kinova_description)/urdf/j2n6s300.xacro"/>
- <xacro:j2n6s300  base_parent="root" prefix="" />
--->
 <env name="GAZEBO_RESOURCE_PATH" value="$(find interbotix_gazebo)"/>
  <xacro:include filename="$(find interbotix_descriptions)/urdf/vx300.urdf.xacro"/>

Commit message: global argument redefinition name_robot to id_robot

File: atom2_common/atom2_description/robots/atom2_std.urdf.xacro (robot description, xacro)
@@ -22,7 +22,7 @@
 -->
 <!-- - - - - - - - - - - - - - GLOBAL ARGUMENTS - - - - - - - - - - - - - -->
-  <xacro:arg name="base_footprint"    default="$(arg robot_name)_base_footprint" />
-  <xacro:arg name="base_link"         default="$(arg robot_name)_base_link" />
-  <xacro:arg name="robot_name"        default="atom2" />
+  <xacro:arg name="base_footprint"    default="$(arg robot_id)_base_footprint" />
+  <xacro:arg name="base_link"         default="$(arg robot_id)_base_link" />
+  <xacro:arg name="robot_id"          default="atom2" />
   <xacro:arg name="use_rplidar_A1M8"  default="true" />
   <xacro:arg name="use_orbbec_astra"  default="true" />
@@ -55,10 +55,10 @@
   <xacro:base_link link_name = "$(arg base_link)" />
   <!-- footprint to base joint -->
-  <xacro:base_footprint_joint prefix = "$(arg robot_name)" parent ="$(arg base_footprint)" child = "$(arg base_link)" >
+  <xacro:base_footprint_joint prefix = "$(arg robot_id)" parent ="$(arg base_footprint)" child = "$(arg base_link)" >
     <origin xyz="0 0 0.213" rpy="0 0 0" />
   </xacro:base_footprint_joint>
   <!-- Cube placed in the rotational center of the robot for debug purposes -->
   <xacro:if value="$(arg use_central_cube)">
-    <xacro:central_cube prefix="$(arg robot_name)" parent ="$(arg base_link)" />
+    <xacro:central_cube prefix="$(arg robot_id)" parent ="$(arg base_link)" />
   </xacro:if>
 <!-- - - - - - - - - - - - - - WHEELS DEFINITION  - - - - - - - - - - - - - -->
@@ -68,14 +68,14 @@
 	<xacro:property name="wheel_offset_z" value="0.10549" />
   <!-- The "prefix" param must end in "right" or "left" to differentiate the wheels in "rubber_wheel" xacro file -->
-  <xacro:rubber_wheel prefix="$(arg robot_name)_rear_right" parent ="$(arg base_link)">
+  <xacro:rubber_wheel prefix="$(arg robot_id)_rear_right" parent ="$(arg base_link)">
   	<origin xyz="-${wheel_offset_x} -${wheel_offset_y} -${wheel_offset_z}" rpy="0 0 0"/>
   </xacro:rubber_wheel>
-  <xacro:rubber_wheel prefix="$(arg robot_name)_rear_left" parent ="$(arg base_link)">
+  <xacro:rubber_wheel prefix="$(arg robot_id)_rear_left" parent ="$(arg base_link)">
   	<origin xyz="-${wheel_offset_x} ${wheel_offset_y} -${wheel_offset_z}" rpy="0 0 0"/>
   </xacro:rubber_wheel>
-  <xacro:rubber_wheel prefix="$(arg robot_name)_front_right" parent ="$(arg base_link)">
+  <xacro:rubber_wheel prefix="$(arg robot_id)_front_right" parent ="$(arg base_link)">
   	<origin xyz="${wheel_offset_x} -${wheel_offset_y} -${wheel_offset_z}" rpy="0 0 0"/>
   </xacro:rubber_wheel>
-  <xacro:rubber_wheel prefix="$(arg robot_name)_front_left" parent ="$(arg base_link)">
+  <xacro:rubber_wheel prefix="$(arg robot_id)_front_left" parent ="$(arg base_link)">
   	<origin xyz="${wheel_offset_x} ${wheel_offset_y} -${wheel_offset_z}" rpy="0 0 0"/>
   </xacro:rubber_wheel>
@@ -83,5 +83,5 @@
   <!-- rplidar A1M8 lidar sensor -->
   <xacro:if value="$(arg use_rplidar_A1M8)">
-    <xacro:sensor_rplidar_A1M8 prefix="$(arg robot_name)_rplidar_A1M8" parent ="$(arg base_link)">
+    <xacro:sensor_rplidar_A1M8 prefix="$(arg robot_id)_rplidar_A1M8" parent ="$(arg base_link)">
       <origin xyz="0.09286 0 0.28275" rpy="0 0 0"/>
     </xacro:sensor_rplidar_A1M8>
@@ -89,8 +89,8 @@
   <!-- kinect camera with support structure -->
   <xacro:if value="$(arg use_kinect)">
-    <xacro:sensor_kinect prefix="$(arg robot_name)_kinect" parent ="$(arg base_link)">
+    <xacro:sensor_kinect prefix="$(arg robot_id)_kinect" parent ="$(arg base_link)">
       <origin xyz="-0.22247 0 0.68823" rpy="0 0 0"/>
     </xacro:sensor_kinect>
-    <xacro:structure_kinect_support prefix="$(arg robot_name)_kinect_support" parent ="$(arg base_link)">
+    <xacro:structure_kinect_support prefix="$(arg robot_id)_kinect_support" parent ="$(arg base_link)">
       <origin xyz="-0.23 0 0.24" rpy="0 0 0"/>
     </xacro:structure_kinect_support>
@@ -98,5 +98,5 @@
   <!-- orbbec astra camera sensor -->
   <xacro:if value="$(arg use_orbbec_astra)">
-    <xacro:sensor_orbbec_astra prefix="$(arg robot_name)_orbbec_astra" parent ="$(arg base_link)">
+    <xacro:sensor_orbbec_astra prefix="$(arg robot_id)_orbbec_astra" parent ="$(arg base_link)">
       <origin xyz="0.31938 0 0.08801" rpy="0 0 0"/>
     </xacro:sensor_orbbec_astra>
@@ -105,45 +105,45 @@
 <env name="GAZEBO_RESOURCE_PATH" value="$(find interbotix_gazebo)"/>
  <xacro:include filename="$(find interbotix_descriptions)/urdf/vx300.urdf.xacro"/>
-  <gazebo reference="$(arg robot_name)/base_link">
+  <gazebo reference="/base_link">
     <material>Custom/Interbotix</material>
   </gazebo>
-  <gazebo reference="$(arg robot_name)/shoulder_link">
+  <gazebo reference="/shoulder_link">
     <material>Custom/Interbotix</material>
   </gazebo>
-  <gazebo reference="$(arg robot_name)/upper_arm_link">
+  <gazebo reference="/upper_arm_link">
     <material>Custom/Interbotix</material>
   </gazebo>
-  <gazebo reference="$(arg robot_name)/forearm_link">
+  <gazebo reference="/forearm_link">
     <material>Custom/Interbotix</material>
   </gazebo>
-  <gazebo reference="$(arg robot_name)/upper_forearm_link">
+  <gazebo reference="/upper_forearm_link">
     <material>Custom/Interbotix</material>
   </gazebo>
-  <gazebo reference="$(arg robot_name)/lower_forearm_link">
+  <gazebo reference="/lower_forearm_link">
     <material>Custom/Interbotix</material>
   </gazebo>
-  <gazebo reference="$(arg robot_name)/wrist_link">
+  <gazebo reference="/wrist_link">
     <material>Custom/Interbotix</material>
   </gazebo>
-  <gazebo reference="$(arg robot_name)/gripper_link">
+  <gazebo reference="/gripper_link">
     <material>Custom/Interbotix</material>
   </gazebo>
-  <gazebo reference="$(arg robot_name)/gripper_prop_link">
+  <gazebo reference="/gripper_prop_link">
     <dampingFactor>1</dampingFactor>
     <material>Custom/Interbotix</material>
   </gazebo>
-  <gazebo reference="$(arg robot_name)/gripper_bar_link">
+  <gazebo reference="/gripper_bar_link">
     <material>Custom/Interbotix</material>
   </gazebo>
-  <gazebo reference="$(arg robot_name)/left_finger_link">
+  <gazebo reference="/left_finger_link">
     <material>Custom/Interbotix</material>
   </gazebo>
-  <gazebo reference="$(arg robot_name)/right_finger_link">
+  <gazebo reference="/right_finger_link">
     <material>Custom/Interbotix</material>
   </gazebo>
     <joint name="arm_base_joint" type="fixed">
 		<origin xyz="0 0 0.21275" rpy="0 0 0" />
-		<parent link="atom2_base_link" />
-		<child link="atom2/base_link" />
+		<parent link="$(arg base_link)" />
+		<child link="/base_link" />
 	  </joint>
 </robot>

Commit message: Implemented xacro macro for vx300 arm

File: atom2_common/atom2_description/robots/atom2_std.urdf.xacro (robot description, xacro)
@@ -22,6 +22,4 @@
 -->
 <!-- - - - - - - - - - - - - - GLOBAL ARGUMENTS - - - - - - - - - - - - - -->
-  <xacro:arg name="base_footprint"    default="$(arg robot_id)_base_footprint" />
-  <xacro:arg name="base_link"         default="$(arg robot_id)_base_link" />
   <xacro:arg name="robot_id"          default="atom2" />
   <xacro:arg name="use_rplidar_A1M8"  default="true" />
@@ -29,4 +27,6 @@
   <xacro:arg name="use_kinect"        default="true" />
   <xacro:arg name="use_central_cube"  default="true" />
+  <xacro:arg name="base_footprint"    default="$(arg robot_id)_base_footprint" />
+  <xacro:arg name="base_link"         default="$(arg robot_id)_base_link" />
 <!-- - - - - - - - - - - - - - XACRO INCLUDES - - - - - - - - - - - - - -->
   <!-- Import atom2 base elements -->
@@ -102,48 +102,8 @@
     </xacro:sensor_orbbec_astra>
   </xacro:if>
-<!-- - - - - - - - - - - - - - UR3 ARM IMPLEMENTATION  - - - - - - - - - - - - - -->
-<env name="GAZEBO_RESOURCE_PATH" value="$(find interbotix_gazebo)"/>
- <xacro:include filename="$(find interbotix_descriptions)/urdf/vx300.urdf.xacro"/>
-  <gazebo reference="/base_link">
-    <material>Custom/Interbotix</material>
-  </gazebo>
-  <gazebo reference="/shoulder_link">
-    <material>Custom/Interbotix</material>
-  </gazebo>
-  <gazebo reference="/upper_arm_link">
-    <material>Custom/Interbotix</material>
-  </gazebo>
-  <gazebo reference="/forearm_link">
-    <material>Custom/Interbotix</material>
-  </gazebo>
-  <gazebo reference="/upper_forearm_link">
-    <material>Custom/Interbotix</material>
-  </gazebo>
-  <gazebo reference="/lower_forearm_link">
-    <material>Custom/Interbotix</material>
-  </gazebo>
-  <gazebo reference="/wrist_link">
-    <material>Custom/Interbotix</material>
-  </gazebo>
-  <gazebo reference="/gripper_link">
-    <material>Custom/Interbotix</material>
-  </gazebo>
-  <gazebo reference="/gripper_prop_link">
-    <dampingFactor>1</dampingFactor>
-    <material>Custom/Interbotix</material>
-  </gazebo>
-  <gazebo reference="/gripper_bar_link">
-    <material>Custom/Interbotix</material>
-  </gazebo>
-  <gazebo reference="/left_finger_link">
-    <material>Custom/Interbotix</material>
-  </gazebo>
-  <gazebo reference="/right_finger_link">
-    <material>Custom/Interbotix</material>
-  </gazebo>
-    <joint name="arm_base_joint" type="fixed">
-		<origin xyz="0 0 0.21275" rpy="0 0 0" />
-		<parent link="$(arg base_link)" />
-		<child link="/base_link" />
-	  </joint>
+<!-- - - - - - - - - - - - - - VX300 ARM IMPLEMENTATION  - - - - - - - - - - - - - -->
+<xacro:include filename="$(find atom2_description)/urdf/accesories/vx300_arm.urdf.xacro" />
+<xacro:vx300_arm parent="$(arg base_link)">
+    <origin xyz="0 0 0.21275" rpy="0 0 0" />
+</xacro:vx300_arm>
 </robot>

Commit message: Modified the origin arm and changed the color arm, now is orange

File: atom2_common/atom2_description/robots/atom2_std.urdf.xacro (robot description, xacro)
@@ -105,5 +105,5 @@
 <xacro:include filename="$(find atom2_description)/urdf/accesories/vx300_arm.urdf.xacro" />
 <xacro:vx300_arm parent="$(arg base_link)">
-    <origin xyz="0 0 0.21275" rpy="0 0 0" />
+    <origin xyz="-0.05 0 0.24" rpy="0 0 0" />
 </xacro:vx300_arm>
 </robot>

File: atom2_common/atom2_description/urdf/accesories/vx300_arm.urdf.xacro (robot description, xacro)
@@ -10,39 +10,39 @@
     </joint>
     <gazebo reference="/base_link">
-      <material>Gazebo/Grey</material>
+      <material>Gazebo/Orange</material>
     </gazebo>
     <gazebo reference="/shoulder_link">
-      <material>Gazebo/Grey</material>
+      <material>Gazebo/Orange</material>
     </gazebo>
     <gazebo reference="/upper_arm_link">
-      <material>Gazebo/Grey</material>
+      <material>Gazebo/Orange</material>
     </gazebo>
     <gazebo reference="/forearm_link">
-      <material>Gazebo/Grey</material>
+      <material>Gazebo/Orange</material>
     </gazebo>
     <gazebo reference="/upper_forearm_link">
-      <material>Gazebo/Grey</material>
+      <material>Gazebo/Orange</material>
     </gazebo>
     <gazebo reference="/lower_forearm_link">
-      <material>Gazebo/Grey</material>
+      <material>Gazebo/Orange</material>
     </gazebo>
     <gazebo reference="/wrist_link">
-      <material>Gazebo/Grey</material>
+      <material>Gazebo/Orange</material>
     </gazebo>
     <gazebo reference="/gripper_link">
-      <material>Gazebo/Grey</material>
+      <material>Gazebo/Orange</material>
     </gazebo>
     <gazebo reference="/gripper_prop_link">
       <dampingFactor>1</dampingFactor>
-      <material>Gazebo/Grey</material>
+      <material>Gazebo/Orange</material>
     </gazebo>
     <gazebo reference="/gripper_bar_link">
-      <material>Gazebo/Grey</material>
+      <material>Gazebo/Orange</material>
     </gazebo>
     <gazebo reference="/left_finger_link">
-      <material>Gazebo/Grey</material>
+      <material>Gazebo/Orange</material>
     </gazebo>
     <gazebo reference="/right_finger_link">
-      <material>Gazebo/Grey</material>
+      <material>Gazebo/Orange</material>
     </gazebo>
   </xacro:macro>

Commit message: Added "use_vx300_arm" argument to launch arm urdf and arm controllers Now, all accesories are set to false by default

File: atom2_common/atom2_description/robots/atom2_std.urdf.xacro (robot description, xacro)
@@ -26,4 +26,5 @@
   <xacro:arg name="use_orbbec_astra"  default="true" />
   <xacro:arg name="use_kinect"        default="true" />
+  <xacro:arg name="use_vx300_arm"     default="true" />
   <xacro:arg name="use_central_cube"  default="true" />
   <xacro:arg name="base_footprint"    default="$(arg robot_id)_base_footprint" />
@@ -103,7 +104,9 @@
   </xacro:if>
 <!-- - - - - - - - - - - - - - VX300 ARM IMPLEMENTATION  - - - - - - - - - - - - - -->
-<xacro:include filename="$(find atom2_description)/urdf/accesories/vx300_arm.urdf.xacro" />
-<xacro:vx300_arm parent="$(arg base_link)">
-    <origin xyz="-0.05 0 0.24" rpy="0 0 0" />
-</xacro:vx300_arm>
+<xacro:if value="$(arg use_vx300_arm)">
+  <xacro:include filename="$(find atom2_description)/urdf/accesories/vx300_arm.urdf.xacro" />
+  <xacro:vx300_arm parent="$(arg base_link)">
+      <origin xyz="-0.05 0 0.24" rpy="0 0 0" />
+  </xacro:vx300_arm>
+</xacro:if>
 </robot>

Commit message: Modified origins

File: atom2_common/atom2_description/robots/atom2_std.urdf.xacro (robot description, xacro)
@@ -23,11 +23,12 @@
 <!-- - - - - - - - - - - - - - GLOBAL ARGUMENTS - - - - - - - - - - - - - -->
   <xacro:arg name="robot_id"          default="atom2" />
-  <xacro:arg name="use_rplidar_A1M8"  default="true" />
-  <xacro:arg name="use_orbbec_astra"  default="true" />
-  <xacro:arg name="use_kinect"        default="true" />
-  <xacro:arg name="use_vx300_arm"     default="true" />
-  <xacro:arg name="use_central_cube"  default="true" />
+  <xacro:arg name="use_rplidar_A1M8"  default="true"  />
+  <xacro:arg name="use_orbbec_astra"  default="true"  />
+  <xacro:arg name="use_kinect"        default="true"  />
+  <xacro:arg name="use_vx300_arm"     default="true"  />
+  <xacro:arg name="use_central_cube"  default="true"  />
   <xacro:arg name="base_footprint"    default="$(arg robot_id)_base_footprint" />
-  <xacro:arg name="base_link"         default="$(arg robot_id)_base_link" />
+  <xacro:arg name="base_link"         default="$(arg robot_id)_base_link"      />
+  <xacro:property name = "M_PI"       value="3.1415926535897931"               />
 <!-- - - - - - - - - - - - - - XACRO INCLUDES - - - - - - - - - - - - - -->
   <!-- Import atom2 base elements -->
@@ -91,8 +92,12 @@
   <xacro:if value="$(arg use_kinect)">
     <xacro:sensor_kinect prefix="$(arg robot_id)_kinect" parent ="$(arg base_link)">
-      <origin xyz="-0.22247 0 0.68823" rpy="0 0 0"/>
+      <!-- <origin xyz="-0.22247 0 0.68823" rpy="0 ${M_PI*0.17} 0"/> -->
+      <!-- <origin xyz="-0.22247 0 0.68823" rpy="0 ${M_PI*0.22} 0"/> -->
+      <!-- <origin xyz="-0.22247 0 0.73" rpy="0 ${M_PI*0.22} 0"/> -->
+      <origin xyz="-0.22247 0 0.75" rpy="0 ${M_PI*0.175} 0"/>
     </xacro:sensor_kinect>
     <xacro:structure_kinect_support prefix="$(arg robot_id)_kinect_support" parent ="$(arg base_link)">
-      <origin xyz="-0.23 0 0.24" rpy="0 0 0"/>
+      <!-- <origin xyz="-0.27 0 0.24" rpy="0 0 0"/> -->
+      <origin xyz="-0.263 0 0.24" rpy="0 0 0"/>
     </xacro:structure_kinect_support>
   </xacro:if>
@@ -107,5 +112,5 @@
   <xacro:include filename="$(find atom2_description)/urdf/accesories/vx300_arm.urdf.xacro" />
   <xacro:vx300_arm parent="$(arg base_link)">
-      <origin xyz="-0.05 0 0.24" rpy="0 0 0" />
+      <origin xyz="-0.04 0 0.24" rpy="0 0 0" />
   </xacro:vx300_arm>
 </xacro:if>
