Commit message: Added new parameters and a function to generate all four wheels

File: atom2_common/atom2_description/urdf/wheels/rubber_wheel.urdf.xacro (robot description, xacro)
@@ -2,5 +2,8 @@
 <robot name="wheels" xmlns:xacro="http://www.ros.org/wiki/xacro">
   <!-- - - - - - - - - - - - - - WHEEL PARAMETERS - - - - - - - - - - - - - -->
-  <xacro:property name = "wheel_mass" value = "2.2" />
+  <xacro:property name = "M_PI"         value="3.1415926535897931" />
+  <xacro:property name = "wheel_mass"   value = "2.2"              />
+  <xacro:property name = "wheel_radius" value = "0.0825"           />
+  <xacro:property name = "wheel_width"  value = "0.045"            />
   <!-- - - - - - - - - - - - - - RIGHT & LEFT INERTIA - - - - - - - - - - - - - -->
   <xacro:macro name="inertia_selector" params = "wheel">
@@ -19,4 +22,13 @@
     <xacro:if value = "${wheel.endswith('left')}">
       <mesh filename="package://atom2_description/meshes/wheels/left_wheel${extension}" />
+    </xacro:if>
+  </xacro:macro>
+  <!-- - - - - - - - - - - - - - RIGHT & LEFT COLLISION - - - - - - - - - - - - - -->
+  <xacro:macro name="origin_collision_selector" params = "wheel">
+    <xacro:if value = "${wheel.endswith('right')}">
+      <origin xyz="0 -0.007 0" rpy="${M_PI/2} 0 0" />
+    </xacro:if>
+    <xacro:if value = "${wheel.endswith('left')}">
+      <origin xyz="0 0.007 0"  rpy="${M_PI/2} 0 0" />
     </xacro:if>
   </xacro:macro>
@@ -44,8 +56,7 @@
       </visual>
       <collision>
-        <origin xyz="0 0 0" rpy="1.57079632679 0 0" />
+        <origin_collision_selector wheel = "${prefix}" />
         <geometry>
-          <!-- <mesh_selector wheel = "${prefix}" extension = "_simple.stl" /> -->
-          <cylinder length="0.04" radius="0.082"/>
+          <cylinder length="${wheel_width}" radius="${wheel_radius}" />
         </geometry>
       </collision>
